File: pcb/hackpad.kicad_pcb (KiCad board)
At the start: 2 copper layers, 83.3 x 61.9 mm, 31 parts, among them U1 XIAO-RP2040-SMD

Commit message: add text and qr code silkscreen
Parts:
- added G***: LOGO, Custom:Github_QR, F.Cu at (35.6, 56.4)
Routing:
- net Row 2: track 103.0 -> 100.5 mm
Other:
- board text added: "Designed by DJ_Laser"
- board text added: "N16-Remote"
- board text added: "https://github.com/dj-laser/n16-remote"
