File: pcb/hackpad.kicad_pcb (KiCad board)
At the start: 2 copper layers, 83.3 x 61.9 mm, 36 parts, among them J1 Conn_01x04_Pin, U1 XIAO-RP2040-SMD

Commit message: add day 1 files
Parts:
- removed D_B1, D_B2, D_B3, D_C1, D_M1, D_M2, D_M3, D_M4, D_R1, D_R2: SK6812MINI, ScottoKeebs_Components:LED_SK6812MINI
- removed G***: LOGO, Custom:Github_QR
- removed REF** (x3): MountingHole_2.2mm_M2, MountingHole:MountingHole_2.2mm_M2
- removed S_B1, S_B2, S_B3, S_C1, S_M1, S_M2, S_M3, S_M4, S_R1, S_R2: Keyswitch, ScottoKeebs_MX:MX_PCB_1.00u
- added D11: Diode, Diode_THT:D_DO-35_SOD27_P7.62mm_Horizontal, F.Cu at (118.4, 102.8)
- added D12: Diode, Diode_THT:D_DO-35_SOD27_P7.62mm_Horizontal, F.Cu at (118.4, 106.3)
- added D13: IR204A, LED_THT:LED_D3.0mm_IRBlack, F.Cu at (197.5, 40.0)
- added J3: OLED_128x32, ScottoKeebs_Components:OLED_128x32, F.Cu at (154.4, 34.8)
- added S_1: Keyswitch, ScottoKeebs_Choc:Choc_V2_1.00u, F.Cu at (162.0, 56.9)
- added S_10: Keyswitch, ScottoKeebs_Choc:Choc_V2_1.00u, F.Cu at (162.0, 107.9)
- added S_11: Keyswitch, ScottoKeebs_Choc:Choc_V2_1.00u, F.Cu at (180.0, 107.9)
- added S_12: Keyswitch, ScottoKeebs_Choc:Choc_V2_1.00u, F.Cu at (198.0, 107.9)
- added S_2: Keyswitch, ScottoKeebs_Choc:Choc_V2_1.00u, F.Cu at (180.0, 56.9)
- added S_3: Keyswitch, ScottoKeebs_Choc:Choc_V2_1.00u, F.Cu at (198.0, 56.9)
- added S_4: Keyswitch, ScottoKeebs_Choc:Choc_V2_1.00u, F.Cu at (162.0, 73.9)
- added S_5: Keyswitch, ScottoKeebs_Choc:Choc_V2_1.00u, F.Cu at (180.0, 73.9)
- added S_6: Keyswitch, ScottoKeebs_Choc:Choc_V2_1.00u, F.Cu at (198.0, 73.9)
- added S_7: Keyswitch, ScottoKeebs_Choc:Choc_V2_1.00u, F.Cu at (162.0, 90.9)
- added S_8: Keyswitch, ScottoKeebs_Choc:Choc_V2_1.00u, F.Cu at (180.0, 90.9)
- added S_9: Keyswitch, ScottoKeebs_Choc:Choc_V2_1.00u, F.Cu at (198.0, 90.9)
- J1: value Conn_01x04_Pin -> Conn_01x03_Pin; footprint Connector_PinHeader_1.00mm:PinHeader_1x04_P1.00mm_Horizontal -> Connector_PinHeader_1.00mm:PinHeader_1x03_P1.00mm_Horizontal
- U1: value XIAO-RP2040-SMD -> RP2040; footprint Seeed Studio XIAO Series Library:XIAO-RP2040-SMD -> Package_DFN_QFN:QFN-56-1EP_7x7mm_P0.4mm_EP3.2x3.2mm; moved to B.Cu
- moved J1 155.0 mm to (203.1, 44.0), turned to 0 degrees
- moved U1 81.3 mm to (181.7, 40.2), turned to 180 degrees
- moved D3 66.6 mm to (118.4, 74.3), turned to 0 degrees
- moved D7 66.2 mm to (118.4, 88.5), turned to 0 degrees
- moved D1 48.1 mm to (118.4, 67.2), turned to 0 degrees
- moved D8 47.2 mm to (118.4, 92.1), turned to 0 degrees
- moved D4 47.1 mm to (118.4, 77.9), turned to 0 degrees
- moved D2 31.1 mm to (118.4, 70.8), turned to 0 degrees
- moved D5 28.5 mm to (118.4, 81.5), turned to 0 degrees
- moved D9 28.1 mm to (118.4, 95.7), turned to 0 degrees
- moved D6 12.5 mm to (118.4, 85.0), turned to 0 degrees
- moved D10 9.77 mm to (118.4, 99.2), turned to 0 degrees
Connections:
- D10 pad 1: Row 2 -> Row 3
- D7 pad 1: Row 1 -> Row 2
- J1 pad 1: Net-(J1-Pin_1) -> unconnected-(J1-Pin_1-Pad1)
- J1 pad 2: Net-(J1-Pin_2) -> unconnected-(J1-Pin_2-Pad2)
- J1 pad 3: Net-(J1-Pin_3) -> unconnected-(J1-Pin_3-Pad3)
- U1 pad 1: unconnected-(U1-GPIO26_A0_D0-Pad1) -> Net-(U1-IOVDD-Pad1)
- U1 pad 10: Col 3 -> Net-(U1-IOVDD-Pad1)
- U1 pad 13: GND -> unconnected-(U1-GPIO10-Pad13)
- U1 pad 14: +5V -> unconnected-(U1-GPIO11-Pad14)
- U1 pad 17: Net-(J1-Pin_1) -> unconnected-(U1-GPIO14-Pad17)
- U1 pad 18: Net-(J1-Pin_2) -> unconnected-(U1-GPIO15-Pad18)
- U1 pad 19: Net-(J1-Pin_3) -> unconnected-(U1-TESTEN-Pad19)
- U1 pad 2: Col 0 -> unconnected-(U1-GPIO0-Pad2)
- U1 pad 20: Net-(J1-Pin_4) -> unconnected-(U1-XIN-Pad20)
- U1 pad 3: RGB -> unconnected-(U1-GPIO1-Pad3)
- U1 pad 4: Row 0 -> unconnected-(U1-GPIO2-Pad4)
- U1 pad 5: Col 2 -> unconnected-(U1-GPIO3-Pad5)
- U1 pad 6: Col 1 -> unconnected-(U1-GPIO4-Pad6)
- U1 pad 8: Row 1 -> unconnected-(U1-GPIO6-Pad8)
- U1 pad 9: Row 2 -> unconnected-(U1-GPIO7-Pad9)
Routing:
- net +5V: track 360.7 -> 0.00 mm, vias 12 -> 0
- net Col 0: track 79.7 -> 0.00 mm
- net Row 1: track 76.2 -> 0.00 mm
- net Row 2: track 72.0 -> 0.00 mm
- net Col 1: track 68.1 -> 0.00 mm, vias 1 -> 0
- net Net-(J1-Pin_2): track 60.5 -> 0.00 mm, vias 1 -> 0
- net Net-(J1-Pin_4): track 59.7 -> 0.00 mm
- net Net-(J1-Pin_1): track 59.2 -> 0.00 mm
- net Net-(J1-Pin_3): track 57.6 -> 0.00 mm
- net Row 0: track 50.7 -> 0.00 mm
- net Col 2: track 48.5 -> 0.00 mm
- net Col 3: track 42.5 -> 0.00 mm
- net Net-(D_C1-DOUT): track 26.8 -> 0.00 mm, vias 2 -> 0
- net Net-(D_B3-DIN): track 23.6 -> 0.00 mm, vias 2 -> 0
- net Net-(D_B1-DOUT): track 19.6 -> 0.00 mm
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- removed copper zone on B.Cu, net GND
- removed copper zone on F.Cu, net GND
Other:
- board outline removed
- board text removed: "Designed by DJ_Laser"
- board text removed: "GND"
- board text removed: "N16-Remote"
- board text removed: "RST"
- board text removed: "SWDCLK"
- board text removed: "SWDIO"
- board text removed: "https://github.com/dj-laser/n16-remote"
