File: pcb/hackpad.kicad_sch (KiCad schematic)
At the start: 32 parts, among them J1 Conn_01x04_Pin, U1 XIAO-RP2040-SMD

Commit message: add day 1 files
Parts:
- removed D6: Diode, Diode_THT:D_DO-35_SOD27_P7.62mm_Horizontal, symbol ScottoKeebs:Placeholder_Diode
- removed D_B1, D_B2, D_B3, D_C1, D_M1, D_M2, D_M3, D_M4, D_R1, D_R2: SK6812MINI, ScottoKeebs_Components:LED_SK6812MINI, symbol ScottoKeebs:LED_SK6812MINI
- removed J1: Conn_01x04_Pin, Connector_PinHeader_1.00mm:PinHeader_1x04_P1.00mm_Horizontal, symbol Connector:Conn_01x04_Pin
- removed S_M4: Keyswitch, ScottoKeebs_MX:MX_PCB_1.00u, symbol ScottoKeebs:Placeholder_Keyswitch
- removed U1: XIAO-RP2040-SMD, Seeed Studio XIAO Series Library:XIAO-RP2040-SMD, symbol Seeed_Studio_XIAO_Series:XIAO-RP2040-SMD
- added D10, D11, D12: Diode, Diode_THT:D_DO-35_SOD27_P7.62mm_Horizontal, symbol ScottoKeebs:Placeholder_Diode
- added D13: IR204A, LED_THT:LED_D3.0mm_IRBlack, symbol LED:IR204A
- added J1: Conn_01x03_Pin, Connector_PinHeader_1.00mm:PinHeader_1x03_P1.00mm_Horizontal, symbol Connector:Conn_01x03_Pin
- added J2: USB_C_Receptacle_USB2.0_14P, symbol Connector:USB_C_Receptacle_USB2.0_14P
- added J3: OLED_128x32, ScottoKeebs_Components:OLED_128x32, symbol ScottoKeebs:OLED_128x32
- added R1, R2: 5.1k, symbol Device:R_Small
- added S_10, S_11, S_12: Keyswitch, ScottoKeebs_Choc:Choc_V2_1.00u, symbol ScottoKeebs:Placeholder_Keyswitch
- added U1: RP2040, Package_DFN_QFN:QFN-56-1EP_7x7mm_P0.4mm_EP3.2x3.2mm, symbol MCU_RaspberryPi:RP2040
- S_1: renamed from S_R1; footprint ScottoKeebs_MX:MX_PCB_1.00u -> ScottoKeebs_Choc:Choc_V2_1.00u
- S_2: renamed from S_C1; footprint ScottoKeebs_MX:MX_PCB_1.00u -> ScottoKeebs_Choc:Choc_V2_1.00u
- S_3: renamed from S_M1; footprint ScottoKeebs_MX:MX_PCB_1.00u -> ScottoKeebs_Choc:Choc_V2_1.00u
- S_4: renamed from S_R2; footprint ScottoKeebs_MX:MX_PCB_1.00u -> ScottoKeebs_Choc:Choc_V2_1.00u
- S_5: renamed from S_M2; footprint ScottoKeebs_MX:MX_PCB_1.00u -> ScottoKeebs_Choc:Choc_V2_1.00u
- S_6: renamed from S_M3; footprint ScottoKeebs_MX:MX_PCB_1.00u -> ScottoKeebs_Choc:Choc_V2_1.00u
- S_7: renamed from S_B3; footprint ScottoKeebs_MX:MX_PCB_1.00u -> ScottoKeebs_Choc:Choc_V2_1.00u
- S_8: renamed from S_B1; footprint ScottoKeebs_MX:MX_PCB_1.00u -> ScottoKeebs_Choc:Choc_V2_1.00u
- S_9: renamed from S_B2; footprint ScottoKeebs_MX:MX_PCB_1.00u -> ScottoKeebs_Choc:Choc_V2_1.00u
- renumbered D3 to D1, D1 to D2, D2 to D3, D7 to D4, D4 to D5, D5 to D6, D10 to D7
Connections:
- net Col 0: now also S_7.1, S_10.1
- net Col 1: now also S_11.1
- net Col 2: now also S_12.1
- net Col 3: no longer S_7.1
- net GND: now also D13.1 (K), J2.A1 (GND), J2.A12 (GND), J2.B1 (GND), J2.B12 (GND), J2.S1 (SHIELD), R1.1, R2.1, U1.57 (GND)
- new net: D10.2 (A), S_10.2
- new net: J2.A5 (CC1), R1.2
- new net: J2.A6 (D+), J2.B6 (D+)
- new net: J2.A7 (D-), J2.B7 (D-)
- new net: J2.B5 (CC2), R2.2
- new net: U1.1 (IOVDD), U1.10 (IOVDD), U1.22 (IOVDD), U1.33 (IOVDD), U1.42 (IOVDD), U1.49 (IOVDD)
- new net: U1.23 (DVDD), U1.50 (DVDD)
- new net: D12.2 (A), S_12.2
- new net: D11.2 (A), S_11.2
- new net Row 3: D10.1 (K), D11.1 (K), D12.1 (K)
- new net USB_D+: U1.47 (USB_DP)
- new net USB_D-: U1.46 (USB_DM)
- new net VBUS: J2.A4 (VBUS), J2.A9 (VBUS), J2.B4 (VBUS), J2.B9 (VBUS)
- no-connect marks 7 -> 0
Other:
- moved on the sheet: D7, S_7
